File: STM32Dimmer.kicad_pcb (KiCad board)
At the start: 2 copper layers, 68.1 x 64.5 mm, 56 parts, among them IC1 CC1101, J1 - Power +, J2 Encoder1, J3 Encoder2, J4 + LED1 -, J5 + LED3 -, J6 + LED5 -, J7 ANT, J8 + LED2 -, J9 + LED4 -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

Commit message: v1.1
Parts:
- added C9: 100n, Capacitors_SMD:C_0805, F.Cu at (188.8, 116.4)
- J1: value - Power + -> Power
- J4: value + LED1 - -> LED1
- J5: value + LED3 - -> LED3
- J6: value + LED5 - -> LED5
- J8: value + LED2 - -> LED2
- J9: value + LED4 - -> LED4
- moved J7 3.77 mm to (192.5, 72.0)
- moved U3 1.59 mm to (191.1, 111.7)
- moved SW1 1.02 mm to (181.6, 72.4), turned to 90 degrees
Connections:
- U4 pad 14: /SW1 -> Net-(U4-Pad14)
- U4 pad 15: /CLK1 -> /PWM4
- U4 pad 16: /DT1 -> /PWM5
- U4 pad 17: Net-(U4-Pad17) -> /SW1
- U4 pad 18: Net-(U4-Pad18) -> /DT1
- U4 pad 19: Net-(U4-Pad19) -> /CLK1
- U4 pad 26: Net-(U4-Pad26) -> /SW2
- U4 pad 35: /DT2 -> Net-(U4-Pad35)
- U4 pad 36: /CLK2 -> Net-(U4-Pad36)
- U4 pad 37: /SW2 -> Net-(U4-Pad37)
- U4 pad 4: /PWM4 -> /CLK2
- U4 pad 5: /PWM5 -> /DT2
Routing:
- net /PWM1: track 81.7 -> 46.6 mm, vias 1 -> 2
- net /SW2: track 19.7 -> 50.1 mm
- net /CLK1: track 42.0 -> 54.6 mm, vias 0 -> 2
- net VCC: track 166.3 -> 175.9 mm, vias 1 -> 2
- net /PWM5: track 34.6 -> 43.3 mm, vias 2 -> 1
- net /DT2: track 17.6 -> 25.6 mm
- net /SW1: track 45.8 -> 53.1 mm, vias 2 -> 1
- net /PWM4: track 41.4 -> 48.3 mm, vias 2 -> 1
- net /CLK2: track 15.8 -> 21.5 mm
- net /SDA: track 32.6 -> 37.8 mm
- net /DT1: track 45.1 -> 49.2 mm, vias 0 -> 2
- net /PWM3: track 16.0 -> 19.2 mm
- net /CSN: track 21.7 -> 24.8 mm
- net Net-(IC1-Pad9): track 3.20 -> 6.30 mm
- net /PWM2: track 20.7 -> 23.5 mm
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- added copper zone on B.Cu, net GND
Other:
- board text added: "STM32 Dimmer V1.1"
- board text removed: "STM32 Dimmer V1.0"

Commit message: small updates / gerber added
Parts:
- J1: value Power -> - Power +
- J4: value LED1 -> + LED1 -
- J5: value LED3 -> + LED3 -
- J6: value LED5 -> + LED5 -
- J8: value LED2 -> + LED2 -
- J9: value LED4 -> + LED4 -
Changed lines of the file:
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@@
     (thickness 1.6)
     (drawings 25)
-    (tracks 430)
+    (tracks 431)
     (zones 0)
     (modules 57)
@@
     (visible_elements 7FFFFFFF)
     (pcbplotparams
-      (layerselection 0x00030_80000001)
-      (usegerberextensions false)
+      (layerselection 0x010fc_80000001)
+      (usegerberextensions true)
       (excludeedgelayer true)
       (linewidth 0.100000)
@@
       (outputformat 1)
       (mirror false)
-      (drillshape 1)
+      (drillshape 0)
       (scaleselection 1)
-      (outputdirectory ""))
+      (outputdirectory gerber/))
   )
   (net 0 "")
@@
       (effects (font (size 1 1) (thickness 0.15)))
     )
-    (fp_text value Power (at 2.794 -5.588 90) (layer F.SilkS)
+    (fp_text value "- Power +" (at 2.794 -5.588 90) (layer F.SilkS)
       (effects (font (size 1 1) (thickness 0.15)))
     )
@@
       (effects (font (size 1 1) (thickness 0.15)))
     )
-    (fp_text value LED1 (at 2.794 -5.588 90) (layer F.SilkS)
+    (fp_text value "+ LED1 -" (at 2.794 -5.588 90) (layer F.SilkS)
       (effects (font (size 1 1) (thickness 0.15)))
     )
@@
       (effects (font (size 1 1) (thickness 0.15)))
     )
-    (fp_text value LED3 (at 2.794 -5.588 90) (layer F.SilkS)
+    (fp_text value "+ LED3 -" (at 2.794 -5.588 90) (layer F.SilkS)
       (effects (font (size 1 1) (thickness 0.15)))
     )
@@
       (effects (font (size 1 1) (thickness 0.15)))
     )
-    (fp_text value LED5 (at 2.54 -5.588 90) (layer F.SilkS)
+    (fp_text value "+ LED5 -" (at 2.54 -5.588 90) (layer F.SilkS)
       (effects (font (size 1 1) (thickness 0.15)))
     )
@@
       (effects (font (size 1 1) (thickness 0.15)))
     )
-    (fp_text value LED2 (at 2.54 -5.588 90) (layer F.SilkS)
+    (fp_text value "+ LED2 -" (at 2.54 -5.588 90) (layer F.SilkS)
       (effects (font (size 1 1) (thickness 0.15)))
     )
@@
       (effects (font (size 1 1) (thickness 0.15)))
     )
-    (fp_text value LED4 (at 2.794 -5.588 90) (layer F.SilkS)
+    (fp_text value "+ LED4 -" (at 2.794 -5.588 90) (layer F.SilkS)
       (effects (font (size 1 1) (thickness 0.15)))
     )
@@
     (effects (font (size 1 1) (thickness 0.15)))
   )
-  (gr_text "STM32 Dimmer\nV1.1" (at 165.608 77.597) (layer F.SilkS)
+  (gr_text "STM32 Dimmer\nV1.1" (at 165.9255 96.7105 90) (layer F.SilkS)
     (effects (font (size 1.2 1.2) (thickness 0.2)))
   )
@@
   (via (at 189.23 118.938) (size 0.6) (drill 0.4) (layers F.Cu B.Cu) (net 32))
   (segment (start 189.738 118.43) (end 189.23 118.938) (width 0.5) (layer B.Cu) (net 32))
+  (segment (start 193.7385 109.2225) (end 195.326 110.81) (width 0.5) (layer B.Cu) (net 33))
+  (segment (start 193.7385 109.2225) (end 175.453 109.2225) (width 0.5) (layer B.Cu) (net 33))
+  (segment (start 175.453 109.2225) (end 174.6885 108.458) (width 0.5) (layer B.Cu) (net 33))
   (segment (start 173.355 86.868) (end 171.8945 88.3285) (width 0.5) (layer F.Cu) (net 33))
   (segment (start 171.8945 88.3285) (end 171.8945 108.458) (width 0.5) (layer F.Cu) (net 33))
-  (segment (start 174.6885 108.458) (end 192.974 108.458) (width 0.5) (layer B.Cu) (net 33))
-  (segment (start 192.974 108.458) (end 195.326 110.81) (width 0.5) (layer B.Cu) (net 33))
   (segment (start 171.8945 108.458) (end 174.6885 108.458) (width 0.25) (layer B.Cu) (net 33))
   (via (at 195.326 110.81) (size 0.6) (drill 0.4) (layers F.Cu B.Cu) (net 33))
